Commit message: Change path

File: kobuki_description/urdf/kobuki.urdf (robot description, URDF)
Before this commit: robot kobuki, 35 links, 34 joints
Links:
- link base_link: geometry collision cylinder length=0.10938 radius=0.178; visual mesh filename=model://kobuki_description/meshes/main_body.dae
- link camera_link: geometry collision box size=0.0730 0.2760 0.0720; visual mesh filename=package://kobuki_description/meshes/sensors/xtion_pro_camer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
- link mount_asus_xtion_pro_link: geometry collision box size=0.0330 0.2760 0.0120; visual mesh filename=package://kobuki_description/meshes/sensors/xtion_pro_stack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
- link plate_bottom_link: geometry collision cylinder length=0.006 radius=0.170; visual mesh filename=package://kobuki_description/meshes/stacks/hexagons/plate_b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
- link plate_middle_link: geometry collision cylinder length=0.006 radius=0.170; visual mesh filename=package://kobuki_description/meshes/stacks/hexagons/plate_m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
- link plate_top_link: geometry collision cylinder length=0.006 radius=0.170; visual mesh filename=package://kobuki_description/meshes/stacks/hexagons/plate_t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
- link standoff_1in_0_link: geometry collision cylinder length=0.0381 radius=0.011113; visual mesh filename=package://kobuki_description/meshes/stacks/circles/68-04552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
- link standoff_1in_1_link: geometry collision cylinder length=0.0381 radius=0.011113; visual mesh filename=package://kobuki_description/meshes/stacks/circles/68-04552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
- link standoff_1in_2_link: geometry collision cylinder length=0.0381 radius=0.011113; visual mesh filename=package://kobuki_description/meshes/stacks/circles/68-04552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
- link standoff_1in_3_link: geometry collision cylinder length=0.0381 radius=0.011113; visual mesh filename=package://kobuki_description/meshes/stacks/circles/68-04552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
- link standoff_1in_4_link: geometry collision cylinder length=0.0381 radius=0.011113; visual mesh filename=package://kobuki_description/meshes/stacks/circles/68-04552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
- link standoff_1in_5_link: geometry collision cylinder length=0.0381 radius=0.011113; visual mesh filename=package://kobuki_description/meshes/stacks/circles/68-04552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
- link standoff_2in_0_link: geometry collision cylinder length=0.0635 radius=0.0381; visual mesh filename=package://kobuki_description/meshes/stacks/circles/68-04552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
- link standoff_2in_1_link: geometry collision cylinder length=0.0635 radius=0.0381; visual mesh filename=package://kobuki_description/meshes/stacks/circles/68-04552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
- link standoff_2in_2_link: geometry collision cylinder length=0.0635 radius=0.0381; visual mesh filename=package://kobuki_description/meshes/stacks/circles/68-04552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
- link standoff_2in_3_link: geometry collision cylinder length=0.0635 radius=0.0381; visual mesh filename=package://kobuki_description/meshes/stacks/circles/68-04552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
- link standoff_8in_0_link: geometry collision cylinder length=0.2032 radius=0.011113; visual mesh filename=package://kobuki_description/meshes/stacks/circles/68-02421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
- link standoff_8in_1_link: geometry collision cylinder length=0.2032 radius=0.011113; visual mesh filename=package://kobuki_description/meshes/stacks/circles/68-02421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
- link standoff_8in_2_link: geometry collision cylinder length=0.2032 radius=0.011113; visual mesh filename=package://kobuki_description/meshes/stacks/circles/68-02421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
- link standoff_8in_3_link: geometry collision cylinder length=0.2032 radius=0.011113; visual mesh filename=package://kobuki_description/meshes/stacks/circles/68-02421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
- link standoff_kinect_0_link: geometry collision cylinder length=0.008585 radius=0.001111; visual mesh filename=package://kobuki_description/meshes/stacks/circles/68-04556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
- link standoff_kinect_1_link: geometry collision cylinder length=0.008585 radius=0.001111; visual mesh filename=package://kobuki_description/meshes/stacks/circles/68-04556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
- link wheel_left_link: geometry collision cylinder length=0.0206 radius=0.035; visual mesh filename=model://kobuki_description/meshes/wheel.dae
- link wheel_right_link: geometry collision cylinder length=0.0206 radius=0.035; visual mesh filename=model://kobuki_description/meshes/wheel.dae
