Commit message: Changed path

File: kobuki_description/urdf/asus_xtion_pro_offset.urdf.xacro (robot description, xacro)
@@ -1,6 +1,6 @@
 <?xml version="1.0"?>
 <robot name="sensor_asus_xtion_pro_offset" xmlns:xacro="http://ros.org/wiki/xacro">
-  <xacro:include filename="$(find kobuki_ros)/urdf/turtlebot_gazebo.urdf.xacro"/>
-  <xacro:include filename="$(find kobuki_ros)/urdf/turtlebot_properties.urdf.xacro"/>
+  <xacro:include filename="$(find kobuki_description)/urdf/turtlebot_gazebo.urdf.xacro"/>
+  <xacro:include filename="$(find kobuki_description)/urdf/turtlebot_properties.urdf.xacro"/>
   <!-- Xacro properties -->
   <xacro:property name="M_SCALE" value="0.001"/>
@@ -33,5 +33,5 @@
         <origin xyz="-0.01 0 0" rpy="${-M_PI/2} -${M_PI} ${-M_PI/2}"/>
         <geometry>
-          <mesh filename="package://kobuki_ros/meshes/sensors/asus_xtion_pro_live.dae" scale="${M_SCALE} ${M_SCALE} ${M_SCALE}"/>
+          <mesh filename="package://kobuki_description/meshes/sensors/asus_xtion_pro_live.dae" scale="${M_SCALE} ${M_SCALE} ${M_SCALE}"/>
         </geometry>
       </visual>

File: kobuki_description/urdf/hexagons.urdf.xacro (robot description, xacro)
@@ -4,5 +4,5 @@
  -->
 <robot name="stack_hexagons" xmlns:xacro="http://ros.org/wiki/xacro">
-  <xacro:include filename="$(find kobuki_ros)/urdf/common_properties.urdf.xacro"/>
+  <xacro:include filename="$(find kobuki_description)/urdf/common_properties.urdf.xacro"/>
   <!-- Xacro properties -->
   <xacro:property name="M_SCALE" value="0.001"/>
@@ -19,5 +19,5 @@
         <origin xyz="0 0 0" rpy="0 0 0"/>
         <geometry>
-          <mesh filename="package://kobuki_ros/meshes/stacks/hexagons/pole_bottom.dae"/>
+          <mesh filename="package://kobuki_description/meshes/stacks/hexagons/pole_bottom.dae"/>
         </geometry>
       </visual>
@@ -47,5 +47,5 @@
         <origin xyz="0 0 0" rpy="0 ${M_PI} 0"/>
         <geometry>
-          <mesh filename="package://kobuki_ros/meshes/stacks/hexagons/pole_middle.dae"/>
+          <mesh filename="package://kobuki_description/meshes/stacks/hexagons/pole_middle.dae"/>
         </geometry>
       </visual>
@@ -75,5 +75,5 @@
         <origin xyz=" 0 0 0" rpy="0 0 0"/>
         <geometry>
-          <mesh filename="package://kobuki_ros/meshes/stacks/hexagons/pole_top.dae"/>
+          <mesh filename="package://kobuki_description/meshes/stacks/hexagons/pole_top.dae"/>
         </geometry>
       </visual>
@@ -103,5 +103,5 @@
         <origin xyz="0 0 -0.01" rpy="0 0 0"/>
         <geometry>
-          <mesh filename="package://kobuki_ros/meshes/sensors/sensor_pole.dae" />
+          <mesh filename="package://kobuki_description/meshes/sensors/sensor_pole.dae" />
         </geometry>
       </visual>
@@ -142,5 +142,5 @@
         <origin xyz="0 0 0" rpy="0 0 0"/>
         <geometry>
-          <mesh filename="package://kobuki_ros/meshes/stacks/hexagons/plate_bottom.dae"/>
+          <mesh filename="package://kobuki_description/meshes/stacks/hexagons/plate_bottom.dae"/>
         </geometry>
       </visual>
@@ -172,5 +172,5 @@
         <origin xyz="0 0 0" rpy="0 0 0"/>
         <geometry>
-          <mesh filename="package://kobuki_ros/meshes/stacks/hexagons/plate_middle.dae"/>
+          <mesh filename="package://kobuki_description/meshes/stacks/hexagons/plate_middle.dae"/>
         </geometry>
       </visual>
@@ -204,5 +204,5 @@
         <origin xyz="0 0 0" rpy="0 0 0"/>
         <geometry>
-          <mesh filename="package://kobuki_ros/meshes/stacks/hexagons/plate_top.dae"/>
+          <mesh filename="package://kobuki_description/meshes/stacks/hexagons/plate_top.dae"/>
         </geometry>
       </visual>

File: kobuki_description/urdf/kobuki.urdf.xacro (robot description, xacro)
@@ -4,9 +4,9 @@
   be incorporated by other urdf files (e.g. turtlebot).
   See kobuki_standalone.urdf.xacro for a standalone urdf to be tested with
-      kobuki_ros/launch/view_model.launch
+      kobuki_description/launch/view_model.launch
  -->
 <robot name="kobuki" xmlns:xacro="http://ros.org/wiki/xacro">
-  <xacro:include filename="$(find kobuki_ros)/urdf/common_properties.urdf.xacro"/>
-  <xacro:include filename="$(find kobuki_ros)/urdf/kobuki_gazebo.urdf.xacro"/>
+  <xacro:include filename="$(find kobuki_description)/urdf/common_properties.urdf.xacro"/>
+  <xacro:include filename="$(find kobuki_description)/urdf/kobuki_gazebo.urdf.xacro"/>
   <!-- Kobuki -->
   <xacro:macro name="kobuki">
@@ -30,5 +30,5 @@
         <geometry>
           <!-- new mesh -->
-          <mesh filename="model://kobuki_ros/meshes/main_body.dae" />
+          <mesh filename="model://kobuki_description/meshes/main_body.dae" />
         </geometry>
         <origin xyz="0.001 0 0.05199" rpy="0 0 0"/>
@@ -65,5 +65,5 @@
       <visual>
         <geometry>
-          <mesh filename="model://kobuki_ros/meshes/wheel.dae"/>
+          <mesh filename="model://kobuki_description/meshes/wheel.dae"/>
         </geometry>
         <origin xyz="0 0 0" rpy="0 0 0"/>
@@ -92,5 +92,5 @@
       <visual>
         <geometry>
-          <mesh filename="model://kobuki_ros/meshes/wheel.dae"/>
+          <mesh filename="model://kobuki_description/meshes/wheel.dae"/>
         </geometry>
         <origin xyz="0 0 0" rpy="0 0 0"/>

File: kobuki_description/urdf/kobuki_hexagons_asus_xtion_pro.urdf.xacro (robot description, xacro)
@@ -6,9 +6,9 @@
 -->
 <robot name="kobuki" xmlns:xacro="http://ros.org/wiki/xacro">
-  <xacro:include filename="$(find kobuki_ros)/urdf/turtlebot_common_library.urdf.xacro" />
-  <xacro:include filename="$(find kobuki_ros)/urdf/kobuki.urdf.xacro" />
-  <xacro:include filename="$(find kobuki_ros)/urdf/stacks/hexagons.urdf.xacro"/>
-  <xacro:include filename="$(find kobuki_ros)/urdf/sensors/asus_xtion_pro.urdf.xacro"/>
-  <xacro:include filename="$(find kobuki_ros)/urdf/stacks/circles.urdf.xacro"/>
+  <xacro:include filename="$(find kobuki_description)/urdf/turtlebot_common_library.urdf.xacro" />
+  <xacro:include filename="$(find kobuki_description)/urdf/kobuki.urdf.xacro" />
+  <xacro:include filename="$(find kobuki_description)/urdf/stacks/hexagons.urdf.xacro"/>
+  <xacro:include filename="$(find kobuki_description)/urdf/sensors/asus_xtion_pro.urdf.xacro"/>
+  <xacro:include filename="$(find kobuki_description)/urdf/stacks/circles.urdf.xacro"/>
   <xacro:kobuki/>
   <xacro:stack_hexagons                 parent="base_link"/>

File: kobuki_description/urdf/kobuki_standalone.urdf.xacro (robot description, xacro)
@@ -6,8 +6,8 @@
        xmlns:xacro="http://ros.org/wiki/xacro">
   <!-- Defines the kobuki component tag. -->
-  <xacro:include filename="$(find kobuki_ros)/urdf/kobuki.urdf.xacro" />
-  <xacro:include filename="$(find kobuki_ros)/urdf/turtlebot_common_library.urdf.xacro" />
-  <xacro:include filename="$(find kobuki_ros)/urdf/stacks/hexagons.urdf.xacro"/>
-  <xacro:include filename="$(find kobuki_ros)/urdf/sensors/asus_xtion_pro.urdf.xacro"/>
+  <xacro:include filename="$(find kobuki_description)/urdf/kobuki.urdf.xacro" />
+  <xacro:include filename="$(find kobuki_description)/urdf/turtlebot_common_library.urdf.xacro" />
+  <xacro:include filename="$(find kobuki_description)/urdf/stacks/hexagons.urdf.xacro"/>
+  <xacro:include filename="$(find kobuki_description)/urdf/sensors/asus_xtion_pro.urdf.xacro"/>
   <xacro:kobuki/>
 </robot>

File: kobuki_description/urdf/sensors/astra.urdf.xacro (robot description, xacro)
@@ -1,6 +1,6 @@
 <?xml version="1.0"?>
 <robot name="sensor_astra" xmlns:xacro="http://ros.org/wiki/xacro">
-  <xacro:include filename="$(find kobuki_ros)/urdf/turtlebot_gazebo.urdf.xacro"/>
-  <xacro:include filename="$(find kobuki_ros)/urdf/turtlebot_properties.urdf.xacro"/>
+  <xacro:include filename="$(find kobuki_description)/urdf/turtlebot_gazebo.urdf.xacro"/>
+  <xacro:include filename="$(find kobuki_description)/urdf/turtlebot_properties.urdf.xacro"/>
   <!-- Xacro properties -->
   <xacro:property name="astra_cam_py" value="-0.0125"/>
@@ -33,5 +33,5 @@
         <origin xyz="-0.04 0.02 -0.01" rpy="${M_PI/2} 0 ${M_PI/2}"/>
         <geometry>
-          <mesh filename="package://kobuki_ros/meshes/sensors/astra.dae" scale="${astra_dae_display_scale} ${astra_dae_display_scale} ${astra_dae_display_scale}"/>
+          <mesh filename="package://kobuki_description/meshes/sensors/astra.dae" scale="${astra_dae_display_scale} ${astra_dae_display_scale} ${astra_dae_display_scale}"/>
         </geometry>
       </visual>

File: kobuki_description/urdf/sensors/asus_xtion_pro.urdf.xacro (robot description, xacro)
@@ -1,6 +1,6 @@
 <?xml version="1.0"?>
 <robot name="sensor_asus_xtion_pro" xmlns:xacro="http://ros.org/wiki/xacro">
-  <xacro:include filename="$(find kobuki_ros)/urdf/turtlebot_gazebo.urdf.xacro"/>
-  <xacro:include filename="$(find kobuki_ros)/urdf/turtlebot_properties.urdf.xacro"/>
+  <xacro:include filename="$(find kobuki_description)/urdf/turtlebot_gazebo.urdf.xacro"/>
+  <xacro:include filename="$(find kobuki_description)/urdf/turtlebot_properties.urdf.xacro"/>
   <!-- Xacro properties -->
   <xacro:property name="M_SCALE" value="0.001"/>
@@ -33,5 +33,5 @@
         <origin xyz="-0.015 0.0035 0.004" rpy="0 0 0"/>
         <geometry>
-          <mesh filename="package://kobuki_ros/meshes/sensors/xtion_pro_camera.dae"/>
+          <mesh filename="package://kobuki_description/meshes/sensors/xtion_pro_camera.dae"/>
         </geometry>
       </visual>
@@ -74,5 +74,5 @@
         <origin xyz="0 0 0" rpy="${-M_PI/2} 0 0"/>
         <geometry>
-          <mesh filename="package://kobuki_ros/meshes/sensors/xtion_pro_stack.dae"/>
+          <mesh filename="package://kobuki_description/meshes/sensors/xtion_pro_stack.dae"/>
         </geometry>
       </visual>

File: kobuki_description/urdf/sensors/kinect.urdf.xacro (robot description, xacro)
@@ -1,6 +1,6 @@
 <?xml version="1.0"?>
 <robot name="sensor_kinect" xmlns:xacro="http://ros.org/wiki/xacro">
-  <xacro:include filename="$(find kobuki_ros)/urdf/turtlebot_gazebo.urdf.xacro"/>
-  <xacro:include filename="$(find kobuki_ros)/urdf/turtlebot_properties.urdf.xacro"/>
+  <xacro:include filename="$(find kobuki_description)/urdf/turtlebot_gazebo.urdf.xacro"/>
+  <xacro:include filename="$(find kobuki_description)/urdf/turtlebot_properties.urdf.xacro"/>
   <xacro:property name="kinect_cam_py" value="-0.0125"/>
   <!-- Parameterised in part by the values in turtlebot_properties.urdf.xacro -->
@@ -27,5 +27,5 @@
        <origin xyz="0 0 0" rpy="0 0 ${M_PI/2}"/>
         <geometry>
-         <mesh filename="package://kobuki_ros/meshes/sensors/kinect.dae"/>
+         <mesh filename="package://kobuki_description/meshes/sensors/kinect.dae"/>
         </geometry>
       </visual>

File: kobuki_description/urdf/sensors/r200.urdf.xacro (robot description, xacro)
@@ -1,6 +1,6 @@
 <?xml version="1.0"?>
 <robot name="sensor_r200" xmlns:xacro="http://ros.org/wiki/xacro">
-  <xacro:include filename="$(find kobuki_ros)/urdf/turtlebot_gazebo.urdf.xacro"/>
-  <xacro:include filename="$(find kobuki_ros)/urdf/turtlebot_properties.urdf.xacro"/>
+  <xacro:include filename="$(find kobuki_description)/urdf/turtlebot_gazebo.urdf.xacro"/>
+  <xacro:include filename="$(find kobuki_description)/urdf/turtlebot_properties.urdf.xacro"/>
   <!-- Mount and camera parameters -->
   <xacro:property name="pole_px" value="-0.103" />
@@ -35,5 +35,5 @@
        <origin xyz="${-r200_bracket_end_width/2} ${r200_bracket_end_offset_py} ${r200_bracket_end_offset_pz}" rpy="0 0 ${-M_PI/2}"/>
         <geometry>
-         <mesh filename="package://kobuki_ros/meshes/sensors/r200_bracket_end.stl" scale="0.001 0.001 0.001"/>
+         <mesh filename="package://kobuki_description/meshes/sensors/r200_bracket_end.stl" scale="0.001 0.001 0.001"/>
         </geometry>
         <xacro:insert_block name="material_dark_grey" />
@@ -50,5 +50,5 @@
        <origin xyz="0 0 0" rpy="0 0 ${M_PI/2}"/>
         <geometry>
-         <mesh filename="package://kobuki_ros/meshes/sensors/r200_bracket.stl" scale="0.001 0.001 0.001"/>
+         <mesh filename="package://kobuki_description/meshes/sensors/r200_bracket.stl" scale="0.001 0.001 0.001"/>
         </geometry>
         <xacro:insert_block name="material_dark_grey" />
@@ -65,5 +65,5 @@
        <origin xyz="${r200_bracket_end_width/2} 0 ${-r200_bracket_end_offset_pz}" rpy="0 0 ${M_PI/2}"/>
         <geometry>
-         <mesh filename="package://kobuki_ros/meshes/sensors/r200_bracket_end.stl" scale="0.001 0.001 0.001"/>
+         <mesh filename="package://kobuki_description/meshes/sensors/r200_bracket_end.stl" scale="0.001 0.001 0.001"/>
         </geometry>
         <xacro:insert_block name="material_dark_grey" />
@@ -80,5 +80,5 @@
        <origin xyz="0 0 0" rpy="${M_PI/2} 0 ${M_PI/2}"/>
         <geometry>
-         <mesh filename="package://kobuki_ros/meshes/sensors/r200.dae" />
+         <mesh filename="package://kobuki_description/meshes/sensors/r200.dae" />
         </geometry>
       </visual>

File: kobuki_description/urdf/stacks/circles.urdf.xacro (robot description, xacro)
@@ -18,5 +18,5 @@
         <origin xyz=" 0 0 0 " rpy="0 0 0" />
         <geometry>
-          <mesh filename="package://kobuki_ros/meshes/stacks/circles/68-02403-125_Spacer.dae"/>
+          <mesh filename="package://kobuki_description/meshes/stacks/circles/68-02403-125_Spacer.dae"/>
         </geometry>
       </visual>
@@ -46,5 +46,5 @@
         <origin xyz=" 0 0 0 " rpy="0 0 0" />
         <geometry>
-          <mesh filename="package://kobuki_ros/meshes/stacks/circles/68-04552-1000-RA_Turtlebot_M-F_Standoff.dae"/>
+          <mesh filename="package://kobuki_description/meshes/stacks/circles/68-04552-1000-RA_Turtlebot_M-F_Standoff.dae"/>
         </geometry>
       </visual>
@@ -74,5 +74,5 @@
         <origin xyz=" 0 0 0 " rpy="0 0 0" />
         <geometry>
-          <mesh filename="package://kobuki_ros/meshes/stacks/circles/68-04552-2000-RA_Turtlebot_M-F_Standoff.dae"/>
+          <mesh filename="package://kobuki_description/meshes/stacks/circles/68-04552-2000-RA_Turtlebot_M-F_Standoff.dae"/>
         </geometry>
       </visual>
@@ -102,5 +102,5 @@
         <origin xyz=" 0 0 0 " rpy="0 0 0" />
         <geometry>
-          <mesh filename="package://kobuki_ros/meshes/stacks/circles/68-02421-8000-RA_Turtlebot_F-F_Standoff.dae"/>
+          <mesh filename="package://kobuki_description/meshes/stacks/circles/68-02421-8000-RA_Turtlebot_F-F_Standoff.dae"/>
         </geometry>
       </visual>
@@ -130,5 +130,5 @@
         <origin xyz=" 0 0 0 " rpy="0 0 0" />
         <geometry>
-          <mesh filename="package://kobuki_ros/meshes/stacks/circles/68-04556-RA_Kinect_Standoff_Assy.dae"/>
+          <mesh filename="package://kobuki_description/meshes/stacks/circles/68-04556-RA_Kinect_Standoff_Assy.dae"/>
         </geometry>
       </visual>
@@ -162,5 +162,5 @@
         <origin xyz=" 0 0 0 " rpy="0 0 0" />
         <geometry>
-          <mesh filename="package://kobuki_ros/meshes/stacks/circles/plate_0_logo.dae"/>
+          <mesh filename="package://kobuki_description/meshes/stacks/circles/plate_0_logo.dae"/>
         </geometry>
       </visual>
@@ -192,5 +192,5 @@
         <origin xyz=" 0 0 0 " rpy="0 0 0" />
         <geometry>
-          <mesh filename="package://kobuki_ros/meshes/stacks/circles/plate_1_logo.dae"/>
+          <mesh filename="package://kobuki_description/meshes/stacks/circles/plate_1_logo.dae"/>
         </geometry>
       </visual>
@@ -222,5 +222,5 @@
         <origin xyz=" 0 0 0 " rpy="0 0 0" />
         <geometry>
-          <mesh filename="package://kobuki_ros/meshes/stacks/circles/plate_1_logo.dae"/>
+          <mesh filename="package://kobuki_description/meshes/stacks/circles/plate_1_logo.dae"/>
         </geometry>
       </visual>
@@ -254,5 +254,5 @@
         <origin xyz=" 0 0 0 " rpy="0 0 0" />
         <geometry>
-          <mesh filename="package://kobuki_ros/meshes/stacks/circles/plate_2_logo.dae"/>
+          <mesh filename="package://kobuki_description/meshes/stacks/circles/plate_2_logo.dae"/>
         </geometry>
       </visual>

File: kobuki_description/urdf/turtlebot_common_library.urdf.xacro (robot description, xacro)
@@ -5,5 +5,5 @@
 <robot xmlns:xacro="http://ros.org/wiki/xacro">
   <!-- General -->
-  <xacro:include filename="$(find kobuki_ros)/urdf/common_properties.urdf.xacro"/>
-  <xacro:include filename="$(find kobuki_ros)/urdf/turtlebot_properties.urdf.xacro"/>
+  <xacro:include filename="$(find kobuki_description)/urdf/common_properties.urdf.xacro"/>
+  <xacro:include filename="$(find kobuki_description)/urdf/turtlebot_properties.urdf.xacro"/>
 </robot>
