Commit message: Fixed bugs with TF in simulation and real

File: kobuki_description/urdf/kobuki_xtion.urdf (robot description, URDF)
Before this commit: robot kobuki, 28 links, 27 joints
Links:
- added link camera_depth_frame
- added link camera_depth_optical_frame
- added link camera_link, mass 0.170; collision box size=0.0730 0.2760 0.0720; visual mesh filename=package://kobuki_description/meshes/sensors/xtion_pro_camer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
- added link camera_rgb_frame
- added link camera_rgb_optical_frame
Joints:
- added joint camera_depth_joint: type fixed, parent camera_rgb_frame, child camera_depth_frame, origin xyz=0 0.027 0 rpy=0 0 0
- added joint camera_depth_optical_joint: type fixed, parent camera_depth_frame, child camera_depth_optical_frame, origin xyz=0 0 0 rpy=-1.5707963267948966 0 -1.5707963267948966
- added joint camera_joint: type fixed, parent camera_rgb_frame, child camera_link, origin xyz=0 -0.022 0 rpy=0 0 0
- added joint camera_rgb_joint: type fixed, parent base_link, child camera_rgb_frame, origin xyz=0.13 0.0205 0.23 rpy=0 0 0
- added joint camera_rgb_optical_joint: type fixed, parent camera_rgb_frame, child camera_rgb_optical_frame, origin xyz=0 0 0 rpy=-1.5707963267948966 0 -1.5707963267948966
