Commit message: Solved TFs

File: kobuki_description/urdf/kobuki_gazebo.urdf (robot description, URDF)
Before this commit: robot kobuki, 36 links, 35 joints
Joints:
- joint camera_depth_optical_joint: origin xyz=0 0 0 rpy=-1.5707963267948966 0 -1.5707963267948966 -> xyz=0 0 0 rpy=0 0 0
- joint camera_rgb_optical_joint: origin xyz=0 0 0 rpy=-1.5707963267948966 0 -1.5707963267948966 -> xyz=0 0 0 rpy=0 0 0

File: kobuki_description/urdf/kobuki_hexagons_asus_xtion_pro.urdf.xacro (robot description, xacro)
@@ -7,5 +7,5 @@
 <robot name="kobuki" xmlns:xacro="http://ros.org/wiki/xacro">
   <xacro:include filename="$(find kobuki_description)/urdf/turtlebot_common_library.urdf.xacro" />
-  <xacro:include filename="$(find kobuki_description)/urdf/kobuki.urdf.xacro" />
+  <xacro:include filename="$(find kobuki_description)/urdf/kobuki_gazebo.urdf.xacro" />
   <xacro:include filename="$(find kobuki_description)/urdf/stacks/hexagons.urdf.xacro"/>
   <xacro:include filename="$(find kobuki_description)/urdf/sensors/asus_xtion_pro.urdf.xacro"/>

File: kobuki_description/urdf/sensors/asus_xtion_pro.urdf.xacro (robot description, xacro)
@@ -18,5 +18,5 @@
     <link name="camera_rgb_frame"/>
     <joint name="camera_rgb_optical_joint" type="fixed">
-      <origin xyz="0 0 0" rpy="${-M_PI/2} 0 ${-M_PI/2}" />
+      <origin xyz="0 0 0" rpy="0 0 0" />
       <parent link="camera_rgb_frame" />
       <child link="camera_rgb_optical_frame" />
@@ -57,5 +57,5 @@
     <link name="camera_depth_frame"/>
     <joint name="camera_depth_optical_joint" type="fixed">
-      <origin xyz="0 0 0" rpy="${-M_PI/2} 0 ${-M_PI/2}" />
+      <origin xyz="0 0 0" rpy="0 0 0" />
       <parent link="camera_depth_frame" />
       <child link="camera_depth_optical_frame" />
